File: PASS ALEPH P 1.7.kicad_pcb (KiCad board)
At the start: 6 copper layers, 200 x 100 mm, 80 parts, among them Q11 BCP56-16,115, Q12 BCP56-16,115, Q2 BCX53-16,115, Q3 IRF610PBF, Q4 IRF610PBF, Q5 IRF9610PBF, Q6 IRF9610PBF, Q7 IRF610PBF, Q8 IRF610PBF, Q9 BCX53-16,115

Commit message: fix some bugs
Routing:
- net Net-(Z1-K): track 41.5 -> 31.4 mm, vias 26 -> 9
- net Net-(Z3-K): track 41.2 -> 31.5 mm, vias 26 -> 9
- net Net-(C3-Pad2): track 58.6 -> 52.9 mm, vias 15 -> 5
- net Net-(C14-Pad1): track 58.5 -> 52.9 mm, vias 15 -> 5
- net Net-(Q5-S): track 40.1 -> 34.5 mm, vias 14 -> 5
- net Net-(Q6-S): track 37.9 -> 33.7 mm, vias 14 -> 5
- net Net-(Z1-A): track 5.88 -> 4.60 mm, vias 12 -> 0
- net Net-(Z3-A): track 5.86 -> 4.60 mm, vias 12 -> 0
- net /IN+: track 6.25 -> 5.93 mm, vias 8 -> 0
- net /IN-: track 6.00 -> 5.93 mm, vias 8 -> 0
- net Net-(Q4-G): track 9.59 -> 9.60 mm, vias 5 -> 0
- net Net-(R19-Pad2): vias 22 -> 14
- net Net-(R18-Pad2): vias 22 -> 14
- net Net-(Q2-E): vias 38 -> 36
- net Net-(Q12-C): vias 13 -> 14
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